File: HARDWARE/EDA/KICAD/pcbcpps/pcbcpps.kicad_pcb (KiCad board)
At the start: 2 copper layers, 57.5 x 39 mm, 20 parts, among them J1 LINE IN, J10 0V, J11 EARTH, J12 EARTH, J2 NEUTRAL, J3 +12V, J4 0V, J5 LINE OUT, J6 LINE OUT, J7 NEUTRAL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

Commit message: adjust conections
Parts:
- moved F1 1.44 mm to (127.0, 92.2)
- turned D1 to 0 degrees
Routing:
- net Net-(F1-Pad2): track 9.27 -> 16.1 mm
- net Net-(D1-Pad2): track 61.2 -> 60.2 mm
Other:
- board size 57.5 x 39 mm -> 57.5 x 38.5 mm
- board text added: "refazer as cotas"
Changed lines of the file:
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@@
   (general
     (thickness 1.6)
-    (drawings 32)
-    (tracks 41)
+    (drawings 35)
+    (tracks 44)
     (zones 0)
     (modules 20)
@@
   )
   (setup
-    (last_trace_width 0.25)
+    (last_trace_width 2)
     (user_trace_width 1.5)
     (user_trace_width 2)
@@
   )
   (module LED_THT:LED_D5.0mm (layer F.Cu)
-    (at 133.8 100.1 90)
+    (at 133.8 100.1)
     (descr "LED, diameter 5.0mm, 2 pins, http://cdn-reichelt.de/documents/datenblatt/A500/LL-504BC2E-009.pdf")
     (tags "LED diameter 5.0mm 2 pins")
-    (fp_text reference D1 (at 1.27 -3.96 90) (layer F.SilkS)
-      (effects (font (size 1 1) (thickness 0.15)))
-    )
-    (fp_text value LED (at 1.27 3.96 90) (layer F.Fab)
-      (effects (font (size 1 1) (thickness 0.15)))
-    )
-    (fp_text user %R (at 1.25 0 90) (layer F.Fab)
+    (fp_text reference D1 (at 1.27 -3.96) (layer F.SilkS)
+      (effects (font (size 1 1) (thickness 0.15)))
+    )
+    (fp_text value LED (at 1.27 3.96) (layer F.Fab)
+      (effects (font (size 1 1) (thickness 0.15)))
+    )
+    (fp_text user %R (at 1.25 0) (layer F.Fab)
       (effects (font (size 0.8 0.8) (thickness 0.2)))
     )
@@
     (fp_arc (start 1.27 0) (end -1.29 -1.54483) (angle 148.9) (layer F.SilkS) (width 0.12))
     (fp_arc (start 1.27 0) (end -1.23 -1.469694) (angle 299.1) (layer F.Fab) (width 0.1))
-    (pad 2 thru_hole circle (at 2.54 0 90) (size 2 2) (drill 0.8) (layers *.Cu *.Mask)
+    (pad 2 thru_hole circle (at 2.54 0) (size 2 2) (drill 0.8) (layers *.Cu *.Mask)
       (net 5 "Net-(D1-Pad2)"))
-    (pad 1 thru_hole rect (at 0 0 90) (size 2 2) (drill 0.8) (layers *.Cu *.Mask)
+    (pad 1 thru_hole rect (at 0 0) (size 2 2) (drill 0.8) (layers *.Cu *.Mask)
       (net 6 "Net-(D1-Pad1)"))
     (model ${KISYS3DMOD}/LED_THT.3dshapes/LED_D5.0mm.wrl
@@
   )
   (module Fuse:Fuseholder_Cylinder-5x20mm_Schurter_0031_8201_Horizontal_Open (layer F.Cu)
-    (at 125.6 91.9 270)
+    (at 127 92.25 270)
     (descr "Fuseholder horizontal open, 5x20mm, 500V, 16A, Schurter 0031.8201, https://us.schurter.com/bundles/snceschurter/epim/_ProdPool_/newDS/en/typ_OGN.pdf")
     (tags "Fuseholder horizontal open 5x20 Schurter 0031.8201")
@@
     )
   )
+  (gr_text "refazer as cotas" (at 150.3 61.9) (layer F.Cu)
+    (effects (font (size 1 1) (thickness 0.15)))
+  )
+  (gr_line (start 176.1 90.7) (end 176.1 78.2) (layer Edge.Cuts) (width 0.1))
+  (gr_line (start 169.1 78.2) (end 176.1 78.2) (layer Edge.Cuts) (width 0.1))
+  (gr_line (start 169.1 90.7) (end 169.1 78.2) (layer Edge.Cuts) (width 0.1))
+  (gr_line (start 166.6 90.7) (end 166.6 78.2) (layer Edge.Cuts) (width 0.1))
+  (gr_line (start 159.6 78.2) (end 166.6 78.2) (layer Edge.Cuts) (width 0.1))
+  (gr_line (start 159.6 90.7) (end 159.6 78.2) (layer Edge.Cuts) (width 0.1))
+  (gr_line (start 157.1 90.7) (end 157.1 78.2) (layer Edge.Cuts) (width 0.1))
+  (gr_line (start 150.1 78.2) (end 157.1 78.2) (layer Edge.Cuts) (width 0.1))
+  (gr_line (start 150.1 90.7) (end 150.1 78.2) (layer Edge.Cuts) (width 0.1))
+  (gr_line (start 147.6 90.7) (end 147.6 78.2) (layer Edge.Cuts) (width 0.1))
+  (gr_line (start 140.6 78.2) (end 147.6 78.2) (layer Edge.Cuts) (width 0.1))
+  (gr_line (start 140.6 90.7) (end 140.6 78.2) (layer Edge.Cuts) (width 0.1))
+  (gr_line (start 138.1 90.7) (end 138.1 78.2) (layer Edge.Cuts) (width 0.1))
+  (gr_line (start 128.6 90.7) (end 128.6 89.7) (layer Edge.Cuts) (width 0.1))
+  (gr_line (start 128.6 90.7) (end 131.1 90.7) (layer Edge.Cuts) (width 0.1))
+  (gr_line (start 176.1 90.7) (end 178.1 90.7) (layer Edge.Cuts) (width 0.1))
+  (gr_line (start 166.6 90.7) (end 169.1 90.7) (layer Edge.Cuts) (width 0.1))
+  (gr_line (start 157.1 90.7) (end 159.6 90.7) (layer Edge.Cuts) (width 0.1))
+  (gr_line (start 147.6 90.7) (end 150.1 90.7) (layer Edge.Cuts) (width 0.1))
   (dimension 39 (width 0.15) (layer Dwgs.User)
     (gr_text "39.000 mm" (at 187.2 97.2 270) (layer Dwgs.User)
@@
     (arrow2b (pts (xy 130.6 71) (xy 131.726504 70.413579)))
   )
-  (gr_line (start 168.6 89.7) (end 168.6 77.7) (layer Edge.Cuts) (width 0.1))
-  (gr_line (start 176.6 77.7) (end 176.6 89.7) (layer Edge.Cuts) (width 0.1))
-  (gr_line (start 138.6 77.7) (end 138.6 89.7) (layer Edge.Cuts) (width 0.1))
-  (gr_line (start 130.6 77.7) (end 138.6 77.7) (layer Edge.Cuts) (width 0.1))
-  (gr_line (start 130.6 89.7) (end 130.6 77.7) (layer Edge.Cuts) (width 0.1))
-  (gr_line (start 130.6 89.7) (end 120.6 89.7) (layer Edge.Cuts) (width 0.1))
+  (gr_line (start 131.1 78.2) (end 138.1 78.2) (layer Edge.Cuts) (width 0.1))
+  (gr_line (start 131.1 90.7) (end 131.1 78.2) (layer Edge.Cuts) (width 0.1))
+  (gr_line (start 128.6 89.7) (end 120.6 89.7) (layer Edge.Cuts) (width 0.1))
   (gr_line (start 120.6 116.7) (end 120.6 89.7) (layer Edge.Cuts) (width 0.1))
   (gr_line (start 178.1 116.7) (end 120.6 116.7) (layer Edge.Cuts) (width 0.1))
-  (gr_line (start 178.1 89.7) (end 178.1 116.7) (layer Edge.Cuts) (width 0.1))
-  (gr_line (start 176.6 89.7) (end 178.1 89.7) (layer Edge.Cuts) (width 0.1))
-  (gr_line (start 168.6 77.7) (end 176.6 77.7) (layer Edge.Cuts) (width 0.1))
-  (gr_line (start 167.1 89.7) (end 168.6 89.7) (layer Edge.Cuts) (width 0.1))
-  (gr_line (start 167.1 77.7) (end 167.1 89.7) (layer Edge.Cuts) (width 0.1))
-  (gr_line (start 159.1 77.7) (end 167.1 77.7) (layer Edge.Cuts) (width 0.1))
-  (gr_line (start 159.1 89.7) (end 159.1 77.7) (layer Edge.Cuts) (width 0.1))
-  (gr_line (start 157.6 89.7) (end 159.1 89.7) (layer Edge.Cuts) (width 0.1))
-  (gr_line (start 157.6 77.7) (end 157.6 89.7) (layer Edge.Cuts) (width 0.1))
-  (gr_line (start 149.6 77.7) (end 157.6 77.7) (layer Edge.Cuts) (width 0.1))
-  (gr_line (start 149.6 89.7) (end 149.6 77.7) (layer Edge.Cuts) (width 0.1))
-  (gr_line (start 148.1 89.7) (end 149.6 89.7) (layer Edge.Cuts) (width 0.1))
-  (gr_line (start 148.1 77.7) (end 148.1 89.7) (layer Edge.Cuts) (width 0.1))
-  (gr_line (start 140.1 77.7) (end 148.1 77.7) (layer Edge.Cuts) (width 0.1))
-  (gr_line (start 140.1 89.7) (end 140.1 77.7) (layer Edge.Cuts) (width 0.1))
-  (gr_line (start 138.6 89.7) (end 140.1 89.7) (layer Edge.Cuts) (width 0.1))
-  (segment (start 127.7 112.1) (end 125.6 114.2) (width 4) (layer B.Cu) (net 1))
-  (segment (start 134 112.1) (end 127.7 112.1) (width 4) (layer B.Cu) (net 1))
+  (gr_line (start 178.1 90.7) (end 178.1 116.7) (layer Edge.Cuts) (width 0.1))
+  (gr_line (start 138.1 90.7) (end 140.6 90.7) (layer Edge.Cuts) (width 0.1))
+  (segment (start 129.65 112.1) (end 127 114.75) (width 3) (layer B.Cu) (net 1))
+  (segment (start 134 112.1) (end 129.65 112.1) (width 3) (layer B.Cu) (net 1))
+  (segment (start 129.34999 112.1) (end 127 114.44999) (width 4) (layer B.Cu) (net 1))
+  (segment (start 134 112.1) (end 129.34999 112.1) (width 4) (layer B.Cu) (net 1))
   (segment (start 144.4 92.5) (end 146.8 92.5) (width 2) (layer B.Cu) (net 2))
   (segment (start 143 93.9) (end 144.4 92.5) (width 2) (layer B.Cu) (net 2))
@@
   (segment (start 174.8 100.9) (end 174.8 106.5) (width 4) (layer B.Cu) (net 4))
   (segment (start 174.8 106.5) (end 172.6 108.7) (width 4) (layer B.Cu) (net 4))
-  (segment (start 125.6 91.9) (end 126.6 92.9) (width 3.5) (layer B.Cu) (net 5))
-  (segment (start 134.6 91.5) (end 134.6 83.7) (width 4) (layer B.Cu) (net 5))
-  (segment (start 133.2 92.9) (end 134.6 91.5) (width 4) (layer B.Cu) (net 5))
-  (segment (start 127 92.9) (end 133.2 92.9) (width 4) (layer B.Cu) (net 5))
   (segment (start 139.2 96.7) (end 135 92.5) (width 2) (layer B.Cu) (net 5))
   (segment (start 140.4 96.7) (end 139.2 96.7) (width 2) (layer B.Cu) (net 5))
-  (segment (start 133.8 93.5) (end 134.8 92.5) (width 2) (layer B.Cu) (net 5))
-  (segment (start 133.8 97.56) (end 133.8 93.5) (width 2) (layer B.Cu) (net 5))
   (segment (start 134.6 93.2) (end 134.6 83.7) (width 4) (layer B.Cu) (net 5))
   (segment (start 138.6 97.2) (end 134.6 93.2) (width 4) (layer B.Cu) (net 5))
@@
   (segment (start 141.4 107.5) (end 138.6 104.7) (width 4) (layer B.Cu) (net 5))
   (segment (start 141.4 112.1) (end 141.4 107.5) (width 4) (layer B.Cu) (net 5))
+  (segment (start 134.6 91.5) (end 134.6 83.7) (width 4) (layer B.Cu) (net 5))
+  (segment (start 133.2 92.9) (end 134.6 91.5) (width 4) (layer B.Cu) (net 5))
+  (segment (start 127.4 92.9) (end 133.2 92.9) (width 4) (layer B.Cu) (net 5))
+  (segment (start 127 92.5) (end 127.4 92.9) (width 4) (layer B.Cu) (net 5))
+  (segment (start 127 92.25) (end 127 92.5) (width 4) (layer B.Cu) (net 5))
+  (segment (start 137 100.1) (end 140.4 96.7) (width 2) (layer B.Cu) (net 5))
+  (segment (start 136.34 100.1) (end 137 100.1) (width 2) (layer B.Cu) (net 5))
   (segment (start 133.8 104.5) (end 133.8 100.1) (width 2) (layer B.Cu) (net 6))
   (segment (start 171.1 104.2) (end 168.6 104.2) (width 1.5) (layer B.Cu) (net 7))

Commit message: adjust pcb
Parts:
- removed J1: LINE IN, TestPoint:TestPoint_Plated_Hole_D5.0mm
- removed J10: 0V, TestPoint:TestPoint_Plated_Hole_D5.0mm
- removed J11, J12: EARTH, TestPoint:TestPoint_Plated_Hole_D5.0mm
- removed J2, J7: NEUTRAL, TestPoint:TestPoint_Plated_Hole_D5.0mm
- removed J5, J6: LINE OUT, TestPoint:TestPoint_Plated_Hole_D5.0mm
- removed J9: +12V, TestPoint:TestPoint_Plated_Hole_D5.0mm
- C1: footprint Capacitor_THT:CP_Radial_D12.5mm_P5.00mm -> Capacitor_THT:CP_Radial_D10.0mm_P5.00mm
- J3: value +12V -> PWR; footprint TestPoint:TestPoint_Plated_Hole_D5.0mm -> Connector_Phoenix_MC_HighVoltage:PhoenixContact_MCV_1,5_2-G-5.08_1x02_P5.08mm_Vertical
- J4: value 0V -> PWR; footprint TestPoint:TestPoint_Plated_Hole_D5.0mm -> Connector_Phoenix_MC_HighVoltage:PhoenixContact_MCV_1,5_4-G-5.08_1x04_P5.08mm_Vertical
- moved J4 25.2 mm to (137.9, 113.2), turned to 0 degrees
- moved J3 6.91 mm to (165.8, 113.3), turned to 0 degrees
- moved R2 6.02 mm to (173.9, 107.0)
- moved R1 4.78 mm to (137.9, 102.0)
- moved D1 4.10 mm to (137.8, 99.5), turned to 90 degrees
- moved D2 3.01 mm to (173.7, 102.7), turned to 180 degrees
- moved F1 2.77 mm to (129.8, 92.6)
- moved RV1 2.75 mm to (143.2, 96.7)
- moved RV2 2.75 mm to (137.6, 92.5)
- moved RV3 2.75 mm to (149.6, 92.5)
- moved C1 0.83 mm to (170.8, 95.8)
Connections:
- C1 pad 2: Net-(C1-Pad2) -> GND
- D1 pad 2: Net-(D1-Pad2) -> /LINE_OUT
- F1 pad 1: Net-(D1-Pad2) -> /LINE_OUT
- J3 pad 1: Net-(C1-Pad1) -> GND
- J4 pad 1: Net-(C1-Pad2) -> Net-(F1-Pad2)
- R1 pad 2: Net-(J2-Pad1) -> Net-(J4-Pad3)
- R2 pad 2: Net-(C1-Pad2) -> GND
- RV1 pad 1: Net-(D1-Pad2) -> /LINE_OUT
- RV1 pad 2: Net-(J11-Pad1) -> Net-(J12-Pad1)
- RV2 pad 1: Net-(D1-Pad2) -> /LINE_OUT
- RV2 pad 2: Net-(J2-Pad1) -> Net-(J4-Pad3)
- RV3 pad 1: Net-(J2-Pad1) -> Net-(J4-Pad3)
- RV3 pad 2: Net-(J11-Pad1) -> Net-(J12-Pad1)
Routing:
- net /LINE_OUT: track 0.00 -> 64.7 mm
- net Net-(D1-Pad2): track 60.2 -> 0.00 mm
- net Net-(J4-Pad3): track 0.00 -> 44.4 mm
- net Net-(J12-Pad1): track 0.00 -> 40.6 mm
- net Net-(J11-Pad1): track 37.6 -> 0.00 mm
- net Net-(J2-Pad1): track 35.5 -> 0.00 mm
- net Net-(C1-Pad2): track 31.0 -> 0.00 mm
- net GND: track 0.00 -> 25.9 mm
- net Net-(C1-Pad1): track 32.4 -> 25.4 mm
- net Net-(F1-Pad2): track 16.1 -> 10.9 mm
- net Net-(D2-Pad1): track 2.50 -> 4.42 mm
- net Net-(D1-Pad1): track 4.40 -> 2.62 mm
Other:
- board size 57.5 x 38.5 mm -> 51.2 x 38.8 mm
- board text removed: "refazer as cotas"
