File: HARDWARE/EDA/KICAD/pcbcpps/pcbcpps.sch (KiCad schematic (older format))
At the start: 20 parts, among them J1 LINE IN, J10 0V, J11 EARTH, J12 EARTH, J2 NEUTRAL, J3 +12V, J4 0V, J5 LINE OUT, J6 LINE OUT, J7 NEUTRAL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

Commit message: adjust pcb
Parts:
- removed J1: LINE IN, TestPoint:TestPoint_Plated_Hole_D5.0mm, symbol Connector:Conn_01x01_Female
- removed J11: EARTH, TestPoint:TestPoint_Plated_Hole_D5.0mm, symbol Connector:Conn_01x01_Female
- removed J2: NEUTRAL, TestPoint:TestPoint_Plated_Hole_D5.0mm, symbol Connector:Conn_01x01_Female
- removed J3: +12V, TestPoint:TestPoint_Plated_Hole_D5.0mm, symbol Connector:Conn_01x01_Female
- removed J4: 0V, TestPoint:TestPoint_Plated_Hole_D5.0mm, symbol Connector:Conn_01x01_Female
- removed J6: LINE OUT, TestPoint:TestPoint_Plated_Hole_D5.0mm, symbol Connector:Conn_01x01_Female
- added J3: PWR, Connector_Phoenix_MC_HighVoltage:PhoenixContact_MCV_1,5_2-G-5.08_1x02_P5.08mm_Vertical, symbol Connector:Screw_Terminal_01x02
- added J4: PWR, Connector_Phoenix_MC_HighVoltage:PhoenixContact_MCV_1,5_4-G-5.08_1x04_P5.08mm_Vertical, symbol Connector:Screw_Terminal_01x04
- C1: footprint Capacitor_THT:CP_Radial_D12.5mm_P5.00mm -> Capacitor_THT:CP_Radial_D10.0mm_P5.00mm
Connections:
- net LINE_OUT: now reaches D1.2 (A), F1.1, J5.1 (Pin_1), RV1.1, RV2.1
- net LINE_OUT: now also J4.2 (Pin_2)
- net at F1.2: now also J4.1 (Pin_1)
- net at J7.1 (Pin_1), R1.2, RV2.2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: now also J4.3 (Pin_3)
- net GND: now reaches C1.2, J10.1 (Pin_1), R2.2
- net GND: now also J3.1 (Pin_1)
- net at C1.1, D2.2 (A), J9.1 (Pin_1): now also J3.2 (Pin_2)
- net at J12.1 (Pin_1), RV1.2, RV3.2: now also J4.4 (Pin_4)
